File: pcb_design/reflexa/reflexa.kicad_sch (KiCad schematic)
At the start: 10 parts, among them J1 Conn_02x13_Odd_Even, J2 USB_C_Receptacle, J3 USB_C_Receptacle, J4 USB_C_Receptacle, J5 USB_C_Receptacle

Commit message: Partial redesign.
Connections:
- net A10-1: now also J1.2 (Pin_2); no longer J1.15 (Pin_15)
- net A10-2: now also J1.10 (Pin_10); no longer J1.8 (Pin_8)
- net A11-1: now also J1.4 (Pin_4); no longer J1.17 (Pin_17)
- net A11-2: now also J1.11 (Pin_11); no longer J1.10 (Pin_10)
- net A2: now also J1.7 (Pin_7); no longer J1.3 (Pin_3)
- net A3-1: now also J1.6 (Pin_6); no longer J1.5 (Pin_5)
- net A3-2: now also J1.13 (Pin_13); no longer J1.2 (Pin_2)
- net A3-3: now also J1.14 (Pin_14); no longer J1.12 (Pin_12)
- net A5-1: now also J1.5 (Pin_5); no longer J1.7 (Pin_7)
- net A5-2: now also J1.12 (Pin_12); no longer J1.4 (Pin_4)
- net A5-3: now also J1.15 (Pin_15); no longer J1.14 (Pin_14)
- net A6: now also J1.8 (Pin_8); no longer J1.9 (Pin_9)
- net A7: now also J1.16 (Pin_16); no longer J1.11 (Pin_11)
- net A8-1: now also J1.3 (Pin_3); no longer J1.13 (Pin_13)
- net A8-2: now also J1.9 (Pin_9); no longer J1.6 (Pin_6)
- net A8-3: now also J1.17 (Pin_17); no longer J1.16 (Pin_16)
Changed lines of the file:
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@@
     (stroke (width 0) (type default) (color 0 0 0 0))
   )
-  (label "A5-3" (at 69.85 146.05 180)
-    (effects (font (size 1.27 1.27)) (justify right bottom))
+  (label "A5-3" (at 40.64 148.59 0)
+    (effects (font (size 1.27 1.27)) (justify left bottom))
   )
   (label "A10-3" (at 193.04 59.69 180)
@@
     (effects (font (size 1.27 1.27)) (justify right bottom))
   )
-  (label "A7" (at 40.64 143.51 0)
-    (effects (font (size 1.27 1.27)) (justify left bottom))
+  (label "A7" (at 69.85 148.59 180)
+    (effects (font (size 1.27 1.27)) (justify right bottom))
   )
   (label "A3-3" (at 193.04 67.31 180)
@@
     (effects (font (size 1.27 1.27)) (justify right bottom))
   )
-  (label "A3-3" (at 69.85 143.51 180)
-    (effects (font (size 1.27 1.27)) (justify right bottom))
-  )
-  (label "A6" (at 40.64 140.97 0)
-    (effects (font (size 1.27 1.27)) (justify left bottom))
-  )
-  (label "A11-1" (at 40.64 151.13 0)
-    (effects (font (size 1.27 1.27)) (justify left bottom))
+  (label "A3-3" (at 69.85 146.05 180)
+    (effects (font (size 1.27 1.27)) (justify right bottom))
+  )
+  (label "A6" (at 69.85 138.43 180)
+    (effects (font (size 1.27 1.27)) (justify right bottom))
+  )
+  (label "A11-1" (at 69.85 133.35 180)
+    (effects (font (size 1.27 1.27)) (justify right bottom))
   )
   (label "A5-3" (at 193.04 41.91 180)
@@
     (effects (font (size 1.27 1.27)) (justify right bottom))
   )
-  (label "A11-2" (at 69.85 140.97 180)
-    (effects (font (size 1.27 1.27)) (justify right bottom))
-  )
-  (label "A8-2" (at 69.85 135.89 180)
-    (effects (font (size 1.27 1.27)) (justify right bottom))
+  (label "A11-2" (at 40.64 143.51 0)
+    (effects (font (size 1.27 1.27)) (justify left bottom))
+  )
+  (label "A8-2" (at 40.64 140.97 0)
+    (effects (font (size 1.27 1.27)) (justify left bottom))
   )
   (label "A3-4" (at 40.64 153.67 0)
@@
     (effects (font (size 1.27 1.27)) (justify right bottom))
   )
-  (label "A10-1" (at 40.64 148.59 0)
-    (effects (font (size 1.27 1.27)) (justify left bottom))
-  )
-  (label "A8-3" (at 69.85 148.59 180)
-    (effects (font (size 1.27 1.27)) (justify right bottom))
+  (label "A10-1" (at 69.85 130.81 180)
+    (effects (font (size 1.27 1.27)) (justify right bottom))
+  )
+  (label "A8-3" (at 40.64 151.13 0)
+    (effects (font (size 1.27 1.27)) (justify left bottom))
   )
   (label "A3-4" (at 247.65 82.55 180)
     (effects (font (size 1.27 1.27)) (justify right bottom))
   )
-  (label "A5-2" (at 69.85 133.35 180)
-    (effects (font (size 1.27 1.27)) (justify right bottom))
-  )
-  (label "A3-2" (at 69.85 130.81 180)
-    (effects (font (size 1.27 1.27)) (justify right bottom))
+  (label "A5-2" (at 69.85 143.51 180)
+    (effects (font (size 1.27 1.27)) (justify right bottom))
+  )
+  (label "A3-2" (at 40.64 146.05 0)
+    (effects (font (size 1.27 1.27)) (justify left bottom))
   )
   (label "A2" (at 193.04 85.09 180)
@@
     (effects (font (size 1.27 1.27)) (justify right bottom))
   )
-  (label "A8-1" (at 40.64 146.05 0)
+  (label "A8-1" (at 40.64 133.35 0)
     (effects (font (size 1.27 1.27)) (justify left bottom))
   )
@@
     (effects (font (size 1.27 1.27)) (justify right bottom))
   )
-  (label "A10-2" (at 69.85 138.43 180)
+  (label "A10-2" (at 69.85 140.97 180)
     (effects (font (size 1.27 1.27)) (justify right bottom))
   )
@@
     (effects (font (size 1.27 1.27)) (justify right bottom))
   )
-  (label "A5-1" (at 40.64 138.43 0)
+  (label "A5-1" (at 40.64 135.89 0)
     (effects (font (size 1.27 1.27)) (justify left bottom))
   )
@@
     (effects (font (size 1.27 1.27)) (justify right bottom))
   )
-  (label "A3-1" (at 40.64 135.89 0)
-    (effects (font (size 1.27 1.27)) (justify left bottom))
+  (label "A3-1" (at 69.85 135.89 180)
+    (effects (font (size 1.27 1.27)) (justify right bottom))
   )
   (label "A11-3" (at 69.85 153.67 180)
@@
     (effects (font (size 1.27 1.27)) (justify right bottom))
   )
-  (label "A2" (at 40.64 133.35 0)
+  (label "A2" (at 40.64 138.43 0)
     (effects (font (size 1.27 1.27)) (justify left bottom))
   )
@@
     )
     (path "/55a8b234-a3b6-469d-a0f7-120a1cd8f2ec"
-      (reference "N1") (unit 1) (value "Housing") (footprint "custom_footprints:Enclosure-Gloxinia2")
-    )
-  )
+      (reference "N1") (unit 1) (value "Housing") (footprint "custom_footprints:Enclosure-Gloxinia_front")
+    )
+  )
