File: pcb_design/reflexa/reflexa.kicad_pcb (KiCad board)
At the start: 2 copper layers, 93 x 73 mm, 10 parts, among them J1 Conn_02x13_Odd_Even, J2 USB_C_Receptacle, J3 USB_C_Receptacle, J4 USB_C_Receptacle, J5 USB_C_Receptacle

Commit message: Partial redesign.
Parts:
- N1: footprint custom_footprints:Enclosure-Gloxinia2 -> custom_footprints:Enclosure-Gloxinia_front
- moved N1 28.0 mm to (147.5, 100.0)
- moved C2 26.0 mm to (138.4, 78.7), turned to 90 degrees
- moved C3 21.0 mm to (146.3, 76.9), turned to 0 degrees
- moved C1 10.1 mm to (158.5, 102.0)
- moved C4 8.30 mm to (168.8, 104.8), turned to 90 degrees
- moved J1 6.00 mm to (133.8, 90.3)
Connections:
- J1 pad 10: /A11-2 -> /A10-2
- J1 pad 11: /A7 -> /A11-2
- J1 pad 12: /A3-3 -> /A5-2
- J1 pad 13: /A8-1 -> /A3-2
- J1 pad 14: /A5-3 -> /A3-3
- J1 pad 15: /A10-1 -> /A5-3
- J1 pad 16: /A8-3 -> /A7
- J1 pad 17: /A11-1 -> /A8-3
- J1 pad 2: /A3-2 -> /A10-1
- J1 pad 3: /A2 -> /A8-1
- J1 pad 4: /A5-2 -> /A11-1
- J1 pad 5: /A3-1 -> /A5-1
- J1 pad 6: /A8-2 -> /A3-1
- J1 pad 7: /A5-1 -> /A2
- J1 pad 8: /A10-2 -> /A6
- J1 pad 9: /A6 -> /A8-2
Routing:
- net /A6: track 171.5 -> 131.5 mm, vias 14 -> 12
- net /A7: track 129.7 -> 99.2 mm, vias 5 -> 4
- net /PS: track 241.6 -> 215.4 mm
- net /A10-1: track 84.2 -> 67.4 mm
- net /A5-1: track 70.1 -> 53.3 mm
- net /A8-1: track 74.1 -> 59.6 mm
- net /A11-1: track 84.9 -> 71.9 mm, vias 4 -> 6
- net /A8-4: track 62.7 -> 50.0 mm, vias 4 -> 5
- net /A10-4: track 70.2 -> 57.7 mm
- net /A8-2: track 61.3 -> 50.5 mm, vias 5 -> 4
- net /A5-3: track 60.8 -> 50.2 mm, vias 5 -> 4
- net /A3-2: track 66.2 -> 56.6 mm, vias 5 -> 4
- net /A11-2: track 65.2 -> 56.1 mm, vias 5 -> 4
- net /A8-3: track 60.3 -> 51.3 mm, vias 5 -> 4
- net /A3-4: track 66.5 -> 58.8 mm, vias 6 -> 4
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Other:
- board size 93 x 73 mm -> 76 x 33 mm

Commit message: Updated files.
Parts:
- moved C2 26.7 mm to (127.2, 102.9)
- moved C3 22.6 mm to (139.4, 98.5), turned to 90 degrees
- moved C1 1.77 mm to (157.8, 103.6)
Routing:
- net GND: track 27.0 -> 36.7 mm, vias 13 -> 18
- net /A2: track 190.3 -> 181.0 mm, vias 19 -> 18
- net /A3-1: track 67.3 -> 62.1 mm
- net /PS: track 215.4 -> 218.4 mm
- net /A10-3: track 62.1 -> 64.7 mm, vias 4 -> 5
- net /A11-1: track 71.9 -> 71.1 mm
- net /A5-1: track 53.3 -> 54.0 mm
- net /A8-3: track 51.3 -> 50.7 mm
- net /A8-1: track 59.6 -> 59.1 mm

Commit message: New and updated board designs.
Routing:
- net /A5-3: track 50.2 -> 49.5 mm
Changed lines of the file:
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@@
   (segment (start 120.57 115.39) (end 121.49 116.31) (width 0.3) (layer "B.Cu") (net 17))
   (segment (start 121.49 116.31) (end 121.96 116.31) (width 0.3) (layer "B.Cu") (net 17))
-  (segment (start 154.5 98.70096) (end 154.25048 98.95048) (width 0.3) (layer "F.Cu") (net 18))
   (segment (start 160 109.75) (end 160 101.5) (width 0.3) (layer "F.Cu") (net 18))
-  (segment (start 154.25048 98.95048) (end 154.24952 98.95048) (width 0.3) (layer "F.Cu") (net 18))
+  (segment (start 153.7 101.45) (end 153.7 94.43) (width 0.3) (layer "F.Cu") (net 18))
+  (segment (start 153.7 94.43) (end 151.555 92.285) (width 0.3) (layer "F.Cu") (net 18))
   (segment (start 156 115) (end 156 116.499071) (width 0.3) (layer "F.Cu") (net 18))
-  (segment (start 153.7 101.45) (end 153.75 101.5) (width 0.3) (layer "F.Cu") (net 18))
-  (segment (start 154.24952 98.95048) (end 153.7 99.5) (width 0.3) (layer "F.Cu") (net 18))
-  (segment (start 151.555 92.285) (end 154.5 95.23) (width 0.3) (layer "F.Cu") (net 18))
   (segment (start 153.75 109) (end 153.75 101.5) (width 0.3) (layer "F.Cu") (net 18))
-  (segment (start 154.5 95.23) (end 154.5 98.70096) (width 0.3) (layer "F.Cu") (net 18))
   (segment (start 154.25 113.75) (end 154.25 109.55997) (width 0.3) (layer "F.Cu") (net 18))
-  (segment (start 153.7 99.5) (end 153.7 101.45) (width 0.3) (layer "F.Cu") (net 18))
   (segment (start 156 116.499071) (end 155.82539 116.673681) (width 0.3) (layer "F.Cu") (net 18))
   (segment (start 159.25 110.5) (end 160 109.75) (width 0.3) (layer "F.Cu") (net 18))
   (segment (start 154.25 109.55997) (end 153.75 109.05997) (width 0.3) (layer "F.Cu") (net 18))
   (segment (start 153.75 109.05997) (end 153.75 109) (width 0.3) (layer "F.Cu") (net 18))
-  (segment (start 151.555 90.275) (end 151.555 92.285) (width 0.3) (layer "F.Cu") (net 18))
+  (segment (start 153.75 101.5) (end 153.7 101.45) (width 0.3) (layer "F.Cu") (net 18))
+  (segment (start 151.555 92.285) (end 151.555 90.275) (width 0.3) (layer "F.Cu") (net 18))
   (via (at 160 101.5) (size 0.8) (drill 0.4) (layers "F.Cu" "B.Cu") (net 18))
   (via (at 155.82539 116.673681) (size 0.8) (drill 0.4) (layers "F.Cu" "B.Cu") (net 18))
