File: pcb_design/planalta/planalta.kicad_sch (KiCad schematic)
At the start: 158 parts, among them J1 USB_C_Receptacle, J2 USB_C_Receptacle, J3 USB_C_Receptacle, J4 USB_C_Receptacle, J5 Conn_02x13_Odd_Even, J6 Conn_02x03_Counter_Clockwise, J9 Conn_01x06_Female, Q1 Q_NMOS_GSD, Q2 Q_NMOS_GSD, Q3 Q_NMOS_GSD, Q4 Q_NMOS_GSD, Q5 Q_NMOS_GSD, SW1 SW_Push, U1 MAX4475_var, U10 dsPIC33EP512MC806, U11 DG2034E, U12 LP2985-5.0, U13 REF2033, U14 OPA320, U15 PGA113, U16 PGA113, U17 TPS737, U18 SiP32431, U19 SiP32431, U2 MAX4475_var, U20 SiP32431, U21 DG2034E, U22 DG2034E, U23 DG2034E, U24 SiP32431, U25 SiP32431, U3 MAX4475_var, U4 MAX4475_var, U5 PGA113, U6 PGA113, U7 MCP2542FD, U8 ADM7170, U9 ADS8332, Y1 Crystal_GND24

Commit message: Update.
Connections:
- net REF_C2 is gone; now on net C1RX: U10.58 (RP96/RF0)
- net C1TX: now also U10.60 (AN24/PWM1L/PMD0/RP80/RE0)
- net CIN1: now also J1.A7 (D-), J1.B7 (D-); no longer J1.A11 (RX2+), J1.B11 (RX1+)
- net CIN2: now also J2.A7 (D-), J2.B7 (D-); no longer J2.A11 (RX2+), J2.B11 (RX1+)
- net CIN3: now also J3.A7 (D-), J3.B7 (D-); no longer J3.A11 (RX2+), J3.B11 (RX1+)
- net CIN4: now also J4.A7 (D-), J4.B7 (D-); no longer J4.A11 (RX2+), J4.B11 (RX1+)
- net EN_VA: now also U10.28 (TDI/AN13/PMA10/RPI45/RB13)
- net OUT1: now also J1.A6 (D+), J1.B6 (D+); no longer J1.A3 (TX1-), J1.B3 (TX2-)
- net OUT2: now also J2.A6 (D+), J2.B6 (D+); no longer J2.A3 (TX1-), J2.B3 (TX2-)
- net OUT3: now also J3.A6 (D+), J3.B6 (D+); no longer J3.A3 (TX1-), J3.B3 (TX2-)
- net OUT4: now also J4.A6 (D+), J4.B6 (D+); no longer J4.A3 (TX1-), J4.B3 (TX2-)
- net SCL1: now also J1.A10 (RX2-), J1.B10 (RX1-), J2.A10 (RX2-), J2.B10 (RX1-); no longer J1.A7 (D-), J1.B7 (D-), J2.A7 (D-), J2.B7 (D-)
- net SCL2: now also J3.A10 (RX2-), J3.B10 (RX1-), J4.A10 (RX2-), J4.B10 (RX1-); no longer J3.A7 (D-), J3.B7 (D-), J4.A7 (D-), J4.B7 (D-)
- net SDA1: now also J1.A3 (TX1-), J1.B3 (TX2-), J2.A3 (TX1-), J2.B3 (TX2-); no longer J1.A6 (D+), J1.B6 (D+), J2.A6 (D+), J2.B6 (D+)
- net SDA2: now also J3.A3 (TX1-), J3.B3 (TX2-), J4.A3 (TX1-), J4.B3 (TX2-); no longer J3.A6 (D+), J3.B6 (D+), J4.A6 (D+), J4.B6 (D+)
- net TERM: now also U10.55 (C3IN1+/RP71/RD7); no longer U10.60 (AN24/PWM1L/PMD0/RP80/RE0)
- net VMID: now also J1.A8 (SBU1), J1.B8 (SBU2), J2.A8 (SBU1), J2.B8 (SBU2), J3.A8 (SBU1), J3.B8 (SBU2), J4.A8 (SBU1), J4.B8 (SBU2); no longer J1.A10 (RX2-), J1.B10 (RX1-), J2.A10 (RX2-), J2.B10 (RX1-), J3.A10 (RX2-), J3.B10 (RX1-), J4.A10 (RX2-), J4.B10 (RX1-)
- net +3V3 renamed +3.3V
- net PGM: no longer names the net of J9.6 (Pin_6)
- no-connect marks 28 -> 34
Other:
- moved on the sheet: C11, C42, C44, J1, J2, J3, U9

Commit message: New and updated board designs.
Parts:
- removed J5: Conn_02x13_Odd_Even, Connector_PinHeader_2.54mm:PinHeader_2x13_P2.54mm_Vertical, symbol Connector_Generic:Conn_02x13_Odd_Even
- removed J6: Conn_02x03_Counter_Clockwise, Connector_PinSocket_2.54mm:PinSocket_2x03_P2.54mm_Vertical, symbol Connector_Generic:Conn_02x03_Counter_Clockwise
- added J5: Conn_02x07_Odd_Even, samtec:SAMTEC_TMMH-107-01-T-DV, symbol Connector_Generic:Conn_02x07_Odd_Even
- N1: footprint custom_footprints:Enclosure-Gloxinia2 -> custom_footprints:Enclosure-Gloxinia4
Connections:
- net +3.3V: now also J5.10 (Pin_10)
- net CAN_C1: now also U10.22 (AN9/PMA7/RPI41/RB9), J5.7 (Pin_7)
- net CAN_C2: now also U10.21 (AN8/PMA6/RPI40/RB8), J5.9 (Pin_9)
- net CAN_H: now also J5.3 (Pin_3)
- net CAN_L: now also J5.5 (Pin_5)
- net GND: now also J5.11 (Pin_11), J5.12 (Pin_12), J5.13 (Pin_13), J5.14 (Pin_14)
- net RX: now also U10.52 (PWMR/RP68/RD4), J5.8 (Pin_8); no longer U10.49 (RP65/RD1)
- net TX: now also U10.51 (PMBE/RP67/RD3), J5.6 (Pin_6); no longer U10.52 (PWMR/RP68/RD4)
- net VBUS: now also J5.1 (Pin_1)
- net ~{CTS}: now also U10.50 (RP66/RD2), J5.4 (Pin_4); no longer U10.51 (PMBE/RP67/RD3)
- net ~{RTS}: now also U10.49 (RP65/RD1), J5.2 (Pin_2); no longer U10.50 (RP66/RD2)
- no-connect marks 34 -> 23
Other:
- moved on the sheet: C10, C12, C22, C29, C30, C33, C34, C36, C38, C4, C68, C69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

Commit message: Expose RTCC pin for synchronisation
Connections:
- net +3.3V: now also J5.12 (Pin_12); no longer J5.10 (Pin_10)
- net GND: no longer J5.12 (Pin_12)
- net RTCC: now reaches U10.42 (RTCC/RPI72/RD8)
- net RTCC: now also J5.10 (Pin_10)
- no-connect marks 23 -> 22
Changed lines of the file:
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@@
   (junction (at 335.534 306.578) (diameter 0) (color 0 0 0 0)
   )
-  (junction (at 543.56 54.61) (diameter 0) (color 0 0 0 0)
-  )
   (junction (at 143.764 265.938) (diameter 0) (color 0 0 0 0)
   )
@@
   (no_connect (at 447.04 255.27))
   (no_connect (at 109.22 142.24))
-  (no_connect (at 152.4 78.74))
   (no_connect (at 152.4 76.2))
   (no_connect (at 91.44 142.24))
@@
     (stroke (width 0) (type default) (color 0 0 0 0))
   )
-  (wire (pts (xy 543.56 52.07) (xy 532.13 52.07))
-    (stroke (width 0) (type default) (color 0 0 0 0))
-  )
   (wire (pts (xy 143.764 269.748) (xy 143.764 265.938))
     (stroke (width 0) (type default) (color 0 0 0 0))
@@
     (stroke (width 0) (type default) (color 0 0 0 0))
   )
-  (wire (pts (xy 543.56 52.07) (xy 543.56 54.61))
-    (stroke (width 0) (type default) (color 0 0 0 0))
-  )
   (wire (pts (xy 352.044 265.938) (xy 345.694 265.938))
     (stroke (width 0) (type default) (color 0 0 0 0))
@@
     (stroke (width 0) (type default) (color 0 0 0 0))
   )
+  (wire (pts (xy 542.29 54.61) (xy 532.13 54.61))
+    (stroke (width 0) (type default) (color 0 0 0 0))
+  )
   (wire (pts (xy 296.164 309.118) (xy 291.084 309.118))
     (stroke (width 0) (type default) (color 0 0 0 0))
@@
     (stroke (width 0) (type default) (color 0 0 0 0))
   )
-  (wire (pts (xy 532.13 46.99) (xy 543.56 46.99))
-    (stroke (width 0) (type default) (color 0 0 0 0))
-  )
   (wire (pts (xy 242.824 385.318) (xy 249.174 385.318))
     (stroke (width 0) (type default) (color 0 0 0 0))
@@
     (stroke (width 0) (type default) (color 0 0 0 0))
   )
+  (wire (pts (xy 152.4 78.74) (xy 161.29 78.74))
+    (stroke (width 0) (type default) (color 0 0 0 0))
+  )
   (wire (pts (xy 480.06 316.23) (xy 488.95 316.23))
     (stroke (width 0) (type default) (color 0 0 0 0))
@@
     (stroke (width 0) (type default) (color 0 0 0 0))
   )
-  (wire (pts (xy 543.56 54.61) (xy 532.13 54.61))
-    (stroke (width 0) (type default) (color 0 0 0 0))
-  )
   (polyline (pts (xy 457.2 119.38) (xy 394.97 119.38))
     (stroke (width 0) (type default) (color 0 0 0 0))
@@
     (stroke (width 0) (type default) (color 0 0 0 0))
   )
+  (wire (pts (xy 532.13 49.53) (xy 542.29 49.53))
+    (stroke (width 0) (type default) (color 0 0 0 0))
+  )
   (wire (pts (xy 242.824 302.768) (xy 252.984 302.768))
     (stroke (width 0) (type default) (color 0 0 0 0))
@@
     (stroke (width 0) (type default) (color 0 0 0 0))
   )
-  (wire (pts (xy 532.13 49.53) (xy 541.02 49.53))
+  (wire (pts (xy 532.13 52.07) (xy 542.29 52.07))
     (stroke (width 0) (type default) (color 0 0 0 0))
   )
@@
     (stroke (width 0) (type default) (color 0 0 0 0))
   )
+  (wire (pts (xy 532.13 46.99) (xy 542.29 46.99))
+    (stroke (width 0) (type default) (color 0 0 0 0))
+  )
   (wire (pts (xy 191.77 88.9) (xy 191.77 90.17))
     (stroke (width 0) (type default) (color 0 0 0 0))
@@
     (effects (font (size 1.27 1.27)) (justify right bottom))
   )
+  (label "RTCC" (at 161.29 78.74 180)
+    (effects (font (size 1.27 1.27)) (justify right bottom))
+  )
   (label "VMID" (at 408.94 303.53 180)
     (effects (font (size 1.27 1.27)) (justify right bottom))
@@
     (effects (font (size 1.27 1.27)) (justify left bottom))
   )
-  (label "RX" (at 543.56 46.99 180)
+  (label "RX" (at 542.29 46.99 180)
     (effects (font (size 1.27 1.27)) (justify right bottom))
   )
@@
     (effects (font (size 1.27 1.27)) (justify left bottom))
   )
+  (label "RTCC" (at 542.29 49.53 180)
+    (effects (font (size 1.27 1.27)) (justify right bottom))
+  )
   (label "DRV2" (at 117.094 309.118 180)
     (effects (font (size 1.27 1.27)) (justify right bottom))
@@
     (pin "2")
   )
-  (symbol (lib_id "power:+3.3V") (at 541.02 49.53 270) (unit 1)
+  (symbol (lib_id "power:+3.3V") (at 542.29 52.07 270) (unit 1)
     (in_bom yes) (on_board yes) (fields_autoplaced)
-    (property "Reference" "#PWR087" (id 0) (at 537.21 49.53 0)
+    (property "Reference" "#PWR087" (id 0) (at 538.48 52.07 0)
       (effects (font (size 1.27 1.27)) hide)
     )
-    (property "Value" "+3.3V" (id 1) (at 544.83 49.5299 90)
+    (property "Value" "+3.3V" (id 1) (at 546.1 52.0699 90)
       (effects (font (size 1.27 1.27)) (justify left))
     )
-    (property "Footprint" "" (id 2) (at 541.02 49.53 0)
+    (property "Footprint" "" (id 2) (at 542.29 52.07 0)
       (effects (font (size 1.27 1.27)) hide)
     )
-    (property "Datasheet" "" (id 3) (at 541.02 49.53 0)
+    (property "Datasheet" "" (id 3) (at 542.29 52.07 0)
       (effects (font (size 1.27 1.27)) hide)
     )
@@
     (pin "2")
   )
-  (symbol (lib_id "power:GND") (at 543.56 54.61 0) (mirror y) (unit 1)
+  (symbol (lib_id "power:GND") (at 542.29 54.61 0) (mirror y) (unit 1)
     (in_bom yes) (on_board yes) (fields_autoplaced)
-    (property "Reference" "#PWR0163" (id 0) (at 543.56 60.96 0)
+    (property "Reference" "#PWR0163" (id 0) (at 542.29 60.96 0)
       (effects (font (size 1.27 1.27)) hide)
     )
-    (property "Value" "GND" (id 1) (at 543.56 59.69 0))
-    (property "Footprint" "" (id 2) (at 543.56 54.61 0)
+    (property "Value" "GND" (id 1) (at 542.29 59.69 0))
+    (property "Footprint" "" (id 2) (at 542.29 54.61 0)
       (effects (font (size 1.27 1.27)) hide)
     )
-    (property "Datasheet" "" (id 3) (at 543.56 54.61 0)
+    (property "Datasheet" "" (id 3) (at 542.29 54.61 0)
       (effects (font (size 1.27 1.27)) hide)
     )

Commit message: Minor improvements.
Mostly related to external pull-ups of 10k for I2C
Parts:
- added R43, R44, R45, R46, R47, R48: 10k, Resistor_SMD:R_0603_1608Metric, symbol Device:R
Connections:
- net +3.3V: now also R43.1, R44.1, R45.1, R46.1, R47.1, R48.1
- net SCL1: now also R43.2
- net SCL2: now also R45.2
- net SDA1: now also R44.2
- net SDA2: now also R46.2
- net ~{INT1}: now also R47.2
- net ~{INT2}: now also R48.2
