File: pcb_design/sylvatica/sylvatica.kicad_pcb (KiCad board)
At the start: 2 copper layers, 93 x 93 mm, 127 parts, among them J1 USB_C_Receptacle, J2 USB_C_Receptacle, J3 USB_C_Receptacle, J4 USB_C_Receptacle, J5 Conn_02x07_Odd_Even, J6 Conn_02x07_Odd_Even, J9 Conn_01x06_Female, Q1 Q_NMOS_GSD, Q2 Q_NMOS_GSD, SW1 SW_Push, U1 PGA113, U10 dsPIC33EP512MC806, U11 SiP32431, U12 LP2985-5.0, U13 REF2033, U14 OPA320, U15 SiP32431, U16 SiP32431, U17 SiP32431, U18 SiP32431, U19 ADM7170, U2 PGA113, U20 MCP2542FD, U21 TPS737, U22 SiP32431, U3 PGA113, U4 PGA113, U5 PGA113, U6 PGA113, U7 PGA113, U8 PGA113, U9 ADS8332, Y1 Crystal_GND24

Commit message: Fix net issue.
Connections:
- C9 pad 1: +5V -> VBUS
- R10 pad 1: +5V -> VBUS
- U12 pad 1: +5V -> VBUS
Routing:
- net VBUS: track 114.2 -> 118.7 mm
- net +5V: track 4.51 -> 0.00 mm

Commit message: Finish rerouting VBUS/5V net
Routing:
- net VBUS: track 118.7 -> 182.2 mm, vias 4 -> 10
- net /EN_VDDA: track 56.6 -> 52.1 mm
- net /PGC: track 30.4 -> 29.6 mm
- net /PGD: track 33.3 -> 32.6 mm
