File: pcb_design/dicio-bcb/dicio-bcb.kicad_pcb (KiCad board)
At the start: 2 copper layers, 93 x 93 mm, 6 parts, among them J1 USB_C_Receptacle, J2 Conn_02x10_Odd_Even, J3 USB_C_Receptacle, J4 USB_C_Receptacle, J5 Conn_01x07

Commit message: Expose RTCC pin for synchronisation
Parts:
- J5: value Conn_01x07 -> Conn_01x08; footprint Connector_PinHeader_2.54mm:PinHeader_1x07_P2.54mm_Vertical -> Connector_PinHeader_2.54mm:PinHeader_1x08_P2.54mm_Vertical
Connections:
- J2 pad 14: GND -> /RTCC
- J5 pad 7: GND -> /RTCC
Routing:
- net /RTCC: track 0.00 -> 42.2 mm
Other:
- board text added: "Gloxinia dicio bottom connector board rev. 2"
- board text added: "RTCC"
- board text removed: "Gloxinia dicio bottom connector board rev. 1"
Changed lines of the file:
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@@
   (net 48 "unconnected-(J4-PadB10)")
   (net 49 "unconnected-(J4-PadB11)")
+  (net 50 "/RTCC")
   (footprint "samtec:SAMTEC-MMS-110-02-X-DV" (layer "F.Cu")
     (at 85 45)
@@
       (net 23 "/U1RX") (pinfunction "Pin_13") (pintype "passive"))
     (pad "14" smd rect locked (at 3 2.654) (size 1.02 2.16) (layers "F.Cu" "F.Paste")
-      (net 1 "GND") (pinfunction "Pin_14") (pintype "passive"))
+      (net 50 "/RTCC") (pinfunction "Pin_14") (pintype "passive"))
     (pad "15" smd rect locked (at 5 -2.654) (size 1.02 2.16) (layers "F.Cu" "F.Paste")
       (net 22 "/U1TX") (pinfunction "Pin_15") (pintype "passive"))
@@
     (pad "" np_thru_hole oval (at -33 -40) (size 3.2 6) (drill oval 3.2 6) (layers F&B.Cu *.Mask))
   )
-  (footprint "Connector_PinHeader_2.54mm:PinHeader_1x07_P2.54mm_Vertical" (layer "F.Cu")
+  (footprint "Connector_PinHeader_2.54mm:PinHeader_1x08_P2.54mm_Vertical" (layer "F.Cu")
     (at 105 55)
-    (descr "Through hole straight pin header, 1x07, 2.54mm pitch, single row")
-    (tags "Through hole pin header THT 1x07 2.54mm single row")
+    (descr "Through hole straight pin header, 1x08, 2.54mm pitch, single row")
+    (tags "Through hole pin header THT 1x08 2.54mm single row")
     (property "Sheetfile" "dicio-bcb.kicad_sch")
     (property "Sheetname" "")
@@
       (effects (font (size 1 1) (thickness 0.15)))
     )
-    (fp_text value "Conn_01x07" (at 0 17.57) (layer "F.Fab")
-      (effects (font (size 1 1) (thickness 0.15)))
-    )
-    (fp_text user "${REFERENCE}" (at 0 7.62 90) (layer "F.Fab")
-      (effects (font (size 1 1) (thickness 0.15)))
-    )
-    (fp_line (start -1.33 1.27) (end -1.33 16.57) (layer "F.SilkS") (width 0.12))
+    (fp_text value "Conn_01x08" (at 0 20.11) (layer "F.Fab")
+      (effects (font (size 1 1) (thickness 0.15)))
+    )
+    (fp_text user "${REFERENCE}" (at 0 8.89 90) (layer "F.Fab")
+      (effects (font (size 1 1) (thickness 0.15)))
+    )
+    (fp_line (start 1.33 1.27) (end 1.33 19.11) (layer "F.SilkS") (width 0.12))
     (fp_line (start -1.33 1.27) (end 1.33 1.27) (layer "F.SilkS") (width 0.12))
-    (fp_line (start 1.33 1.27) (end 1.33 16.57) (layer "F.SilkS") (width 0.12))
+    (fp_line (start -1.33 19.11) (end 1.33 19.11) (layer "F.SilkS") (width 0.12))
     (fp_line (start -1.33 0) (end -1.33 -1.33) (layer "F.SilkS") (width 0.12))
+    (fp_line (start -1.33 1.27) (end -1.33 19.11) (layer "F.SilkS") (width 0.12))
     (fp_line (start -1.33 -1.33) (end 0 -1.33) (layer "F.SilkS") (width 0.12))
-    (fp_line (start -1.33 16.57) (end 1.33 16.57) (layer "F.SilkS") (width 0.12))
-    (fp_line (start -1.8 -1.8) (end -1.8 17.05) (layer "F.CrtYd") (width 0.05))
-    (fp_line (start 1.8 17.05) (end 1.8 -1.8) (layer "F.CrtYd") (width 0.05))
+    (fp_line (start -1.8 -1.8) (end -1.8 19.55) (layer "F.CrtYd") (width 0.05))
+    (fp_line (start -1.8 19.55) (end 1.8 19.55) (layer "F.CrtYd") (width 0.05))
+    (fp_line (start 1.8 19.55) (end 1.8 -1.8) (layer "F.CrtYd") (width 0.05))
     (fp_line (start 1.8 -1.8) (end -1.8 -1.8) (layer "F.CrtYd") (width 0.05))
-    (fp_line (start -1.8 17.05) (end 1.8 17.05) (layer "F.CrtYd") (width 0.05))
-    (fp_line (start 1.27 -1.27) (end 1.27 16.51) (layer "F.Fab") (width 0.1))
-    (fp_line (start 1.27 16.51) (end -1.27 16.51) (layer "F.Fab") (width 0.1))
+    (fp_line (start -1.27 -0.635) (end -0.635 -1.27) (layer "F.Fab") (width 0.1))
+    (fp_line (start 1.27 -1.27) (end 1.27 19.05) (layer "F.Fab") (width 0.1))
+    (fp_line (start 1.27 19.05) (end -1.27 19.05) (layer "F.Fab") (width 0.1))
+    (fp_line (start -1.27 19.05) (end -1.27 -0.635) (layer "F.Fab") (width 0.1))
     (fp_line (start -0.635 -1.27) (end 1.27 -1.27) (layer "F.Fab") (width 0.1))
-    (fp_line (start -1.27 16.51) (end -1.27 -0.635) (layer "F.Fab") (width 0.1))
-    (fp_line (start -1.27 -0.635) (end -0.635 -1.27) (layer "F.Fab") (width 0.1))
     (pad "1" thru_hole rect (at 0 0) (size 1.7 1.7) (drill 1) (layers *.Cu *.Mask)
       (net 18 "/~{U1RTS}") (pinfunction "Pin_1") (pintype "passive"))
@@
       (net 25 "/SYNC") (pinfunction "Pin_6") (pintype "passive"))
     (pad "7" thru_hole oval (at 0 15.24) (size 1.7 1.7) (drill 1) (layers *.Cu *.Mask)
-      (net 1 "GND") (pinfunction "Pin_7") (pintype "passive"))
-    (model "${KICAD6_3DMODEL_DIR}/Connector_PinHeader_2.54mm.3dshapes/PinHeader_1x07_P2.54mm_Vertical.wrl"
+      (net 50 "/RTCC") (pinfunction "Pin_7") (pintype "passive"))
+    (pad "8" thru_hole oval (at 0 17.78) (size 1.7 1.7) (drill 1) (layers *.Cu *.Mask)
+      (net 1 "GND") (pinfunction "Pin_8") (pintype "passive"))
+    (model "${KICAD6_3DMODEL_DIR}/Connector_PinHeader_2.54mm.3dshapes/PinHeader_1x08_P2.54mm_Vertical.wrl"
       (offset (xyz 0 0 0))
       (scale (xyz 1 1 1))
@@
     (effects (font (size 1 1) (thickness 0.25)) (justify left))
   )
-  (gr_text "Gloxinia\ndicio bottom connector board\nrev. 1" (at 45 60) (layer "F.SilkS")
+  (gr_text "Gloxinia\ndicio bottom connector board\nrev. 2" (at 45 60) (layer "F.SilkS")
     (effects (font (size 1.5 1.5) (thickness 0.3)) (justify left))
   )
-  (gr_text "GND" (at 107 70) (layer "F.SilkS")
+  (gr_text "GND" (at 107 73) (layer "F.SilkS")
     (effects (font (size 1 1) (thickness 0.25)) (justify left))
   )
   (gr_text "TX" (at 107 60) (layer "F.SilkS")
+    (effects (font (size 1 1) (thickness 0.25)) (justify left))
+  )
+  (gr_text "RTCC" (at 107 70) (layer "F.SilkS")
     (effects (font (size 1 1) (thickness 0.25)) (justify left))
   )
@@
   (segment (start 93.5 129.09) (end 95.09 129.09) (width 0.3) (layer "B.Cu") (net 28))
   (segment (start 105.425 129.8) (end 107.838071 129.8) (width 0.3) (layer "B.Cu") (net 28))
+  (segment (start 100.025 44.65) (end 88.8 44.65) (width 0.3) (layer "F.Cu") (net 50))
+  (segment (start 88.8 44.65) (end 88 45.45) (width 0.3) (layer "F.Cu") (net 50))
+  (segment (start 105 70.24) (end 102.2 67.44) (width 0.3) (layer "F.Cu") (net 50))
+  (segment (start 88 45.45) (end 88 47.654) (width 0.3) (layer "F.Cu") (net 50))
+  (segment (start 102.2 67.44) (end 102.2 46.825) (width 0.3) (layer "F.Cu") (net 50))
+  (segment (start 102.2 46.825) (end 100.025 44.65) (width 0.3) (layer "F.Cu") (net 50))
   (zone (net 1) (net_name "GND") (layer "F.Cu") (hatch edge 0.508)
     (connect_pads (clearance 0.508))
