File: pcb_design/sylvatica-tcb/sylvatica-tcb.kicad_sch (KiCad schematic)
At the start: 6 parts, among them J1 Conn_02x07_Odd_Even, J2 USB_C_Receptacle, J3 USB_C_Receptacle, J4 USB_C_Receptacle, J5 USB_C_Receptacle

Commit message: Gerber exports
Connections:
- no-connect marks 16 -> 24
Changed lines of the file:
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@@
   )
   (no_connect (at 165.1 115.57))
+  (no_connect (at 217.17 77.47))
+  (no_connect (at 67.31 78.74))
+  (no_connect (at 165.1 80.01))
   (no_connect (at 115.57 101.6))
   (no_connect (at 67.31 132.08))
@@
   (no_connect (at 217.17 100.33))
   (no_connect (at 67.31 116.84))
+  (no_connect (at 115.57 81.28))
   (no_connect (at 165.1 128.27))
+  (no_connect (at 67.31 81.28))
+  (no_connect (at 217.17 80.01))
   (no_connect (at 217.17 115.57))
   (no_connect (at 115.57 116.84))
   (no_connect (at 67.31 129.54))
+  (no_connect (at 165.1 77.47))
   (no_connect (at 217.17 128.27))
   (no_connect (at 165.1 130.81))
+  (no_connect (at 115.57 78.74))
   (no_connect (at 165.1 100.33))
   (no_connect (at 217.17 130.81))
@@
     (pin "S1")
   )
+  (symbol (lib_id "power:GND") (at 99.06 30.48 0) (unit 1)
+    (in_bom yes) (on_board yes) (fields_autoplaced)
+    (property "Reference" "#PWR06" (id 0) (at 99.06 36.83 0)
+      (effects (font (size 1.27 1.27)) hide)
+    )
+    (property "Value" "GND" (id 1) (at 99.06 35.56 0))
+    (property "Footprint" "" (id 2) (at 99.06 30.48 0)
+      (effects (font (size 1.27 1.27)) hide)
+    )
+    (property "Datasheet" "" (id 3) (at 99.06 30.48 0)
+      (effects (font (size 1.27 1.27)) hide)
+    )
+    (pin "1")
+  )
   (symbol (lib_id "power:GND") (at 146.05 138.43 0) (unit 1)
     (in_bom yes) (on_board yes) (fields_autoplaced)
@@
     )
     (property "Datasheet" "" (id 3) (at 198.12 138.43 0)
+      (effects (font (size 1.27 1.27)) hide)
+    )
+    (pin "1")
+  )
+  (symbol (lib_id "power:PWR_FLAG") (at 99.06 30.48 0) (unit 1)
+    (in_bom yes) (on_board yes) (fields_autoplaced)
+    (property "Reference" "#FLG01" (id 0) (at 99.06 28.575 0)
+      (effects (font (size 1.27 1.27)) hide)
+    )
+    (property "Value" "PWR_FLAG" (id 1) (at 99.06 25.4 0))
+    (property "Footprint" "" (id 2) (at 99.06 30.48 0)
+      (effects (font (size 1.27 1.27)) hide)
+    )
+    (property "Datasheet" "~" (id 3) (at 99.06 30.48 0)
       (effects (font (size 1.27 1.27)) hide)
     )
@@
   )
   (symbol_instances
+    (path "/e5587b07-bbfc-4184-85ee-e8b978f4103a"
+      (reference "#FLG01") (unit 1) (value "PWR_FLAG") (footprint "")
+    )
     (path "/cf8952af-6e54-4726-9eab-9fbd61f77f85"
       (reference "#PWR01") (unit 1) (value "GND") (footprint "")
@@
       (reference "#PWR05") (unit 1) (value "GND") (footprint "")
     )
+    (path "/99a7c2b9-9c1d-4814-a3da-7b2ae41ed9f6"
+      (reference "#PWR06") (unit 1) (value "GND") (footprint "")
+    )
     (path "/556bddaf-808a-439c-8271-052a1e5d13c2"

Commit message: Various updates for Aisler order.
Parts:
- J1: MPN (none) -> TMMH-107-01-T-DV; Manufacturer (none) -> Samtec
- J2, J3, J4, J5: MPN (none) -> 124018612112A; Manufacturer (none) -> Amphenol
Changed lines of the file:
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@@
+      (effects (font (size 1.27 1.27)) hide)
+    )
+    (property "MPN" "124018612112A" (id 4) (at 201.93 97.79 0)
+      (effects (font (size 1.27 1.27)) hide)
+    )
+    (property "Manufacturer" "Amphenol" (id 5) (at 201.93 97.79 0)
       (effects (font (size 1.27 1.27)) hide)
     )
@@
       (effects (font (size 1.27 1.27)) hide)
     )
+    (property "MPN" "TMMH-107-01-T-DV" (id 4) (at 39.37 36.83 0)
+      (effects (font (size 1.27 1.27)) hide)
+    )
+    (property "Manufacturer" "Samtec" (id 5) (at 39.37 36.83 0)
+      (effects (font (size 1.27 1.27)) hide)
+    )
     (pin "1")
     (pin "10")
@@
     )
     (property "Datasheet" "https://www.usb.org/sites/default/files/documents/usb_type-c.zip" (id 3) (at 55.88 99.06 0)
+      (effects (font (size 1.27 1.27)) hide)
+    )
+    (property "MPN" "124018612112A" (id 4) (at 52.07 99.06 0)
+      (effects (font (size 1.27 1.27)) hide)
+    )
+    (property "Manufacturer" "Amphenol" (id 5) (at 52.07 99.06 0)
       (effects (font (size 1.27 1.27)) hide)
     )
@@
       (effects (font (size 1.27 1.27)) hide)
     )
+    (property "MPN" "124018612112A" (id 4) (at 100.33 99.06 0)
+      (effects (font (size 1.27 1.27)) hide)
+    )
+    (property "Manufacturer" "Amphenol" (id 5) (at 100.33 99.06 0)
+      (effects (font (size 1.27 1.27)) hide)
+    )
     (pin "A1")
     (pin "A10")
@@
       (effects (font (size 1.27 1.27)) hide)
     )
+    (property "MPN" "124018612112A" (id 4) (at 149.86 97.79 0)
+      (effects (font (size 1.27 1.27)) hide)
+    )
+    (property "Manufacturer" "Amphenol" (id 5) (at 149.86 97.79 0)
+      (effects (font (size 1.27 1.27)) hide)
+    )
