File: pcb_design/dicio/dicio.kicad_sch (KiCad schematic)
At the start: 78 parts, among them J1 Conn_02x10_Odd_Even, J2 Conn_01x06_Female, J3 USB_C_Receptacle, J4 Micro_SD_Card, J5 USB_C_Receptacle, J6 USB_C_Receptacle, J8 USB_C_Receptacle, Q1 Q_NMOS_GSD, SW1 SW_SPST, SW2 SW_SPST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

Commit message: Various updates for Aisler order.
Parts:
- removed Y1: Crystal_GND24, Crystal:Crystal_SMD_Abracon_ABM3B-4Pin_5.0x3.2mm, symbol Device:Crystal_GND24
- added Y1: Crystal, Crystal:Crystal_SMD_3215-2Pin_3.2x1.5mm, symbol Device:Crystal
- C21, C22: Mouser (none) -> 80-C1206C475K4PAC
- C29, C6: value 20pF -> 22pF; Mouser 603-CC603FRNPO9BN100 -> 80-C0603C220J3HACTU
- C7, C8: value 20pF -> 30pF; Mouser 603-CC603FRNPO9BN100 -> 80-C0603C300G1HACTU
- J3, J5, J6, J8: Mouser (none) -> 523-124018612112A
Connections:
- net SOSC1: now also Y1.2
- net SOSC2: now also Y1.1
Changed lines of the file:
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@@
     (in_bom yes) (on_board yes)
     (property "Reference" "C7" (id 0) (at 225.552 21.0312 90))
-    (property "Value" "20pF" (id 1) (at 225.552 23.3426 90))
+    (property "Value" "30pF" (id 1) (at 225.552 23.3426 90))
     (property "Footprint" "Capacitor_SMD:C_0603_1608Metric" (id 2) (at 221.742 28.3972 0)
       (effects (font (size 1.27 1.27)) hide)
@@
       (effects (font (size 1.27 1.27)) hide)
     )
-    (property "Mouser" "603-CC603FRNPO9BN100" (id 4) (at 144.272 -377.698 0)
+    (property "Mouser" "80-C0603C300G1HACTU" (id 4) (at 144.272 -377.698 0)
       (effects (font (size 1.27 1.27)) hide)
     )
@@
     (in_bom yes) (on_board yes)
     (property "Reference" "C8" (id 0) (at 225.552 41.402 90))
-    (property "Value" "20pF" (id 1) (at 225.552 43.942 90))
+    (property "Value" "30pF" (id 1) (at 225.552 43.942 90))
     (property "Footprint" "Capacitor_SMD:C_0603_1608Metric" (id 2) (at 221.742 38.5572 0)
       (effects (font (size 1.27 1.27)) hide)
@@
       (effects (font (size 1.27 1.27)) hide)
     )
-    (property "Mouser" "603-CC603FRNPO9BN100" (id 4) (at 134.112 -367.538 0)
+    (property "Mouser" "80-C0603C300G1HACTU" (id 4) (at 134.112 -367.538 0)
       (effects (font (size 1.27 1.27)) hide)
     )
@@
     (pin "1")
   )
-  (symbol (lib_id "Device:Crystal_GND24") (at 182.372 32.512 90) (unit 1)
-    (in_bom yes) (on_board yes)
-    (property "Reference" "Y1" (id 0) (at 188.4934 31.3436 90)
-      (effects (font (size 1.27 1.27)) (justify right))
-    )
-    (property "Value" "Crystal_GND24" (id 1) (at 188.4934 33.655 90)
-      (effects (font (size 1.27 1.27)) (justify right))
-    )
-    (property "Footprint" "Crystal:Crystal_SMD_Abracon_ABM3B-4Pin_5.0x3.2mm" (id 2) (at 182.372 32.512 0)
-      (effects (font (size 1.27 1.27)) hide)
-    )
-    (property "Datasheet" "~" (id 3) (at 182.372 32.512 0)
-      (effects (font (size 1.27 1.27)) hide)
-    )
-    (property "Mouser" "520-.327-12.5-17X-CT" (id 4) (at 182.372 32.512 90)
-      (effects (font (size 1.27 1.27)) hide)
-    )
-    (property "Price" "0.796" (id 5) (at 182.372 32.512 90)
-      (effects (font (size 1.27 1.27)) hide)
-    )
-    (pin "1")
-    (pin "2")
-    (pin "3")
-    (pin "4")
-  )
   (symbol (lib_id "custom_components:TPS737") (at 60.96 78.74 0) (unit 1)
     (in_bom yes) (on_board yes)
@@
     (pin "1")
   )
-  (symbol (lib_id "power:GND") (at 177.292 32.512 270) (unit 1)
-    (in_bom yes) (on_board yes)
-    (property "Reference" "#PWR0132" (id 0) (at 170.942 32.512 0)
-      (effects (font (size 1.27 1.27)) hide)
-    )
-    (property "Value" "GND" (id 1) (at 174.0408 32.639 90)
-      (effects (font (size 1.27 1.27)) (justify right))
-    )
-    (property "Footprint" "" (id 2) (at 177.292 32.512 0)
-      (effects (font (size 1.27 1.27)) hide)
-    )
-    (property "Datasheet" "" (id 3) (at 177.292 32.512 0)
-      (effects (font (size 1.27 1.27)) hide)
-    )
-    (pin "1")
-  )
-  (symbol (lib_id "power:GND") (at 187.452 32.512 90) (unit 1)
-    (in_bom yes) (on_board yes)
-    (property "Reference" "#PWR0133" (id 0) (at 193.802 32.512 0)
-      (effects (font (size 1.27 1.27)) hide)
-    )
-    (property "Value" "GND" (id 1) (at 190.7032 32.385 90)
-      (effects (font (size 1.27 1.27)) (justify right))
-    )
-    (property "Footprint" "" (id 2) (at 187.452 32.512 0)
-      (effects (font (size 1.27 1.27)) hide)
-    )
-    (property "Datasheet" "" (id 3) (at 187.452 32.512 0)
-      (effects (font (size 1.27 1.27)) hide)
-    )
-    (pin "1")
-  )
   (symbol (lib_id "Device:C") (at 187.452 27.432 270) (unit 1)
     (in_bom yes) (on_board yes)
     (property "Reference" "C6" (id 0) (at 187.452 21.0312 90))
-    (property "Value" "20pF" (id 1) (at 187.452 23.3426 90))
+    (property "Value" "22pF" (id 1) (at 187.452 23.3426 90))
     (property "Footprint" "Capacitor_SMD:C_0603_1608Metric" (id 2) (at 183.642 28.3972 0)
       (effects (font (size 1.27 1.27)) hide)
@@
       (effects (font (size 1.27 1.27)) hide)
     )
-    (property "Mouser" "603-CC603FRNPO9BN100" (id 4) (at 106.172 -377.698 0)
+    (property "Mouser" "80-C0603C220J3HACTU" (id 4) (at 106.172 -377.698 0)
       (effects (font (size 1.27 1.27)) hide)
     )
@@
     (in_bom yes) (on_board yes)
     (property "Reference" "C29" (id 0) (at 187.452 41.402 90))
-    (property "Value" "20pF" (id 1) (at 187.452 43.942 90))
+    (property "Value" "22pF" (id 1) (at 187.452 43.942 90))
     (property "Footprint" "Capacitor_SMD:C_0603_1608Metric" (id 2) (at 183.642 38.5572 0)
       (effects (font (size 1.27 1.27)) hide)
@@
       (effects (font (size 1.27 1.27)) hide)
     )
-    (property "Mouser" "603-CC603FRNPO9BN100" (id 4) (at 96.012 -367.538 0)
+    (property "Mouser" "80-C0603C220J3HACTU" (id 4) (at 96.012 -367.538 0)
       (effects (font (size 1.27 1.27)) hide)
     )
@@
       (effects (font (size 1.27 1.27)) hide)
     )
+    (property "Mouser" "80-C1206C475K4PAC" (id 4) (at 36.83 36.83 0)
+      (effects (font (size 1.27 1.27)) hide)
+    )
     (pin "1")
     (pin "2")
@@
       (effects (font (size 1.27 1.27)) hide)
     )
+    (property "Mouser" "80-C1206C475K4PAC" (id 4) (at 86.36 36.83 0)
+      (effects (font (size 1.27 1.27)) hide)
+    )
     (pin "1")
     (pin "2")
@@
       (effects (font (size 1.27 1.27)) hide)
     )
+    (property "Mouser" "523-124018612112A " (id 4) (at 430.53 146.05 0)
+      (effects (font (size 1.27 1.27)) hide)
+    )
     (pin "A1")
     (pin "A10")
@@
       (effects (font (size 1.27 1.27)) hide)
     )
+    (property "Mouser" "523-124018612112A " (id 4) (at 430.53 62.23 0)
+      (effects (font (size 1.27 1.27)) hide)
+    )
     (pin "A1")
     (pin "A10")
@@
       (effects (font (size 1.27 1.27)) hide)
     )
+    (property "Mouser" "523-124018612112A " (id 4) (at 504.19 63.5 0)
+      (effects (font (size 1.27 1.27)) hide)
+    )
     (pin "A1")
     (pin "A10")
@@
     (pin "S1")
   )
+  (symbol (lib_id "Device:Crystal") (at 182.372 32.512 90) (unit 1)
+    (in_bom yes) (on_board yes) (fields_autoplaced)
+    (property "Reference" "Y1" (id 0) (at 186.182 31.2419 90)
+      (effects (font (size 1.27 1.27)) (justify right))
+    )
+    (property "Value" "Crystal" (id 1) (at 186.182 33.7819 90)
+      (effects (font (size 1.27 1.27)) (justify right))
+    )
+    (property "Footprint" "Crystal:Crystal_SMD_3215-2Pin_3.2x1.5mm" (id 2) (at 182.372 32.512 0)
+      (effects (font (size 1.27 1.27)) hide)
+    )
+    (property "Datasheet" "~" (id 3) (at 182.372 32.512 0)
+      (effects (font (size 1.27 1.27)) hide)
+    )
+    (property "Mouser" "520-.327-9-34QCNT" (id 4) (at 182.372 32.512 90)
+      (effects (font (size 1.27 1.27)) hide)
+    )
+    (pin "1")
+    (pin "2")
+  )
   (symbol (lib_id "power:+3.3V") (at 204.47 152.4 90) (unit 1)
     (in_bom yes) (on_board yes)
@@
       (effects (font (size 1.27 1.27)) hide)
     )
+    (property "Mouser" "523-124018612112A " (id 4) (at 504.19 146.05 0)
+      (effects (font (size 1.27 1.27)) hide)
+    )
     (pin "A1")
     (pin "A10")
@@
       (reference "#PWR0131") (unit 1) (value "GND") (footprint "")
     )
-    (path "/00000000-0000-0000-0000-000062c89f09"
-      (reference "#PWR0132") (unit 1) (value "GND") (footprint "")
-    )
-    (path "/00000000-0000-0000-0000-000062c89f13"
-      (reference "#PWR0133") (unit 1) (value "GND") (footprint "")
-    )
     (path "/00000000-0000-0000-0000-000062c89f35"
       (reference "#PWR0134") (unit 1) (value "GND") (footprint "")
@@
     )
     (path "/00000000-0000-0000-0000-000062c89f1f"
-      (reference "C6") (unit 1) (value "20pF") (footprint "Capacitor_SMD:C_0603_1608Metric")
+      (reference "C6") (unit 1) (value "22pF") (footprint "Capacitor_SMD:C_0603_1608Metric")
     )
     (path "/00000000-0000-0000-0000-00005bff6f49"
-      (reference "C7") (unit 1) (value "20pF") (footprint "Capacitor_SMD:C_0603_1608Metric")
+      (reference "C7") (unit 1) (value "30pF") (footprint "Capacitor_SMD:C_0603_1608Metric")
     )
     (path "/00000000-0000-0000-0000-00005bff7020"
-      (reference "C8") (unit 1) (value "20pF") (footprint "Capacitor_SMD:C_0603_1608Metric")
+      (reference "C8") (unit 1) (value "30pF") (footprint "Capacitor_SMD:C_0603_1608Metric")
     )
     (path "/00000000-0000-0000-0000-00005c0ac1f6"
@@
     )
     (path "/00000000-0000-0000-0000-000062c89f2b"
-      (reference "C29") (unit 1) (value "20pF") (footprint "Capacitor_SMD:C_0603_1608Metric")
+      (reference "C29") (unit 1) (value "22pF") (footprint "Capacitor_SMD:C_0603_1608Metric")
     )
     (path "/00000000-0000-0000-0000-00006234ebec"
@@
       (reference "U8") (unit 1) (value "FT232RL") (footprint "Package_SO:SSOP-28_5.3x10.2mm_P0.65mm")
     )
-    (path "/00000000-0000-0000-0000-00005c83da83"
-      (reference "Y1") (unit 1) (value "Crystal_GND24") (footprint "Crystal:Crystal_SMD_Abracon_ABM3B-4Pin_5.0x3.2mm")
+    (path "/98913f12-c757-41c6-8231-39620ab398e7"
+      (reference "Y1") (unit 1) (value "Crystal") (footprint "Crystal:Crystal_SMD_3215-2Pin_3.2x1.5mm")
     )
     (path "/00000000-0000-0000-0000-000062c89f4b"

Commit message: Updates
Connections:
- net AS2: now also J6.A7 (D-), J6.B7 (D-), U1.63 (AN27PWM2H/PMD3/RPI83/RE3); no longer J5.A7 (D-), J5.B7 (D-), U1.14 (AN2/C2IN2-/VMIO/RPI34/RB2)
- net AS3: now also J5.A7 (D-), J5.B7 (D-), U1.14 (AN2/C2IN2-/VMIO/RPI34/RB2); no longer J6.A7 (D-), J6.B7 (D-), U1.63 (AN27PWM2H/PMD3/RPI83/RE3)
- net OW2: now also J6.A6 (D+), J6.B6 (D+), U1.3 (AN31/PWM4H/PMD7/RP87/RE7); no longer J5.A6 (D+), J5.B6 (D+), U1.13 (AN3/C2IN1+/VPIO/RPI35/RB3)
- net OW3: now also J5.A6 (D+), J5.B6 (D+), U1.13 (AN3/C2IN1+/VPIO/RPI35/RB3); no longer J6.A6 (D+), J6.B6 (D+), U1.3 (AN31/PWM4H/PMD7/RP87/RE7)
- net SCL1: now also J3.A10 (RX2-), J3.B10 (RX1-), J6.A10 (RX2-), J6.B10 (RX1-), R13.2, U1.44 (ASCL1/PMCS2/RPI74/RD10); no longer J5.A10 (RX2-), J5.B10 (RX1-), J8.A10 (RX2-), J8.B10 (RX1-), R15.2, U1.32 (SCL2/PMA8/RP101/RF5)
- net SCL2: now also J5.A10 (RX2-), J5.B10 (RX1-), J8.A10 (RX2-), J8.B10 (RX1-), R15.2, U1.32 (SCL2/PMA8/RP101/RF5); no longer J3.A10 (RX2-), J3.B10 (RX1-), J6.A10 (RX2-), J6.B10 (RX1-), R13.2, U1.44 (ASCL1/PMCS2/RPI74/RD10)
- net SDA1: now also J3.A3 (TX1-), J3.B3 (TX2-), J6.A3 (TX1-), J6.B3 (TX2-), R12.2, U1.43 (ASDA1/RPI73/RD9); no longer J5.A3 (TX1-), J5.B3 (TX2-), J8.A3 (TX1-), J8.B3 (TX2-), R14.2, U1.31 (SDA2/PMA9/RP100/RF4)
- net SDA2: now also J5.A3 (TX1-), J5.B3 (TX2-), J8.A3 (TX1-), J8.B3 (TX2-), R14.2, U1.31 (SDA2/PMA9/RP100/RF4); no longer J3.A3 (TX1-), J3.B3 (TX2-), J6.A3 (TX1-), J6.B3 (TX2-), R12.2, U1.43 (ASDA1/RPI73/RD9)
- net ~{INT1}: now also J3.A2 (TX1+), J3.B2 (TX2+), J6.A2 (TX1+), J6.B2 (TX2+), R24.2, U1.62 (AN26/PWM2L/PMD2/RP82/RE2); no longer J5.A2 (TX1+), J5.B2 (TX2+), J8.A2 (TX1+), J8.B2 (TX2+), R22.2, U1.12 (AN4/C1IN2-/RPI36/RB4)
- net ~{INT2}: now also J5.A2 (TX1+), J5.B2 (TX2+), J8.A2 (TX1+), J8.B2 (TX2+), R22.2, U1.12 (AN4/C1IN2-/RPI36/RB4); no longer J3.A2 (TX1+), J3.B2 (TX2+), J6.A2 (TX1+), J6.B2 (TX2+), R24.2, U1.62 (AN26/PWM2L/PMD2/RP82/RE2)
