File: pcb_design/hirsuta/hirsuta.kicad_sch (KiCad schematic)
At the start: 31 parts, among them J1 Screw_Terminal_01x08, J2 Screw_Terminal_01x11, U1 ADS1219, U2 ADP7142AUJZ-1.8

Commit message: Updates
Parts:
- C10, C11, C12, C9: value C -> 0.1uF
- R3, R4, R5, R6: value R -> 1k
Changed lines of the file:
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@@
       (effects (font (size 1.27 1.27)) (justify left))
     )
-    (property "Value" "C" (id 1) (at 118.618 117.0939 0)
+    (property "Value" "0.1uF" (id 1) (at 118.618 117.0939 0)
       (effects (font (size 1.27 1.27)) (justify left))
     )
@@
     (in_bom yes) (on_board yes) (fields_autoplaced)
     (property "Reference" "R6" (id 0) (at 110.49 113.284 90))
-    (property "Value" "R" (id 1) (at 110.49 115.824 90))
+    (property "Value" "1k" (id 1) (at 110.49 115.824 90))
     (property "Footprint" "Capacitor_SMD:C_0603_1608Metric" (id 2) (at 110.49 121.412 90)
       (effects (font (size 1.27 1.27)) hide)
@@
       (effects (font (size 1.27 1.27)) (justify left))
     )
-    (property "Value" "C" (id 1) (at 186.436 132.0799 0)
+    (property "Value" "0.1uF" (id 1) (at 186.436 132.0799 0)
       (effects (font (size 1.27 1.27)) (justify left))
     )
@@
     (in_bom yes) (on_board yes) (fields_autoplaced)
     (property "Reference" "R5" (id 0) (at 178.308 128.27 90))
-    (property "Value" "R" (id 1) (at 178.308 130.81 90))
+    (property "Value" "1k" (id 1) (at 178.308 130.81 90))
     (property "Footprint" "Capacitor_SMD:C_0603_1608Metric" (id 2) (at 178.308 136.398 90)
       (effects (font (size 1.27 1.27)) hide)
@@
     (in_bom yes) (on_board yes) (fields_autoplaced)
     (property "Reference" "R4" (id 0) (at 110.236 124.46 90))
-    (property "Value" "R" (id 1) (at 110.236 127 90))
+    (property "Value" "1k" (id 1) (at 110.236 127 90))
     (property "Footprint" "Capacitor_SMD:C_0603_1608Metric" (id 2) (at 110.236 132.588 90)
       (effects (font (size 1.27 1.27)) hide)
@@
     (in_bom yes) (on_board yes) (fields_autoplaced)
     (property "Reference" "R3" (id 0) (at 178.054 139.446 90))
-    (property "Value" "R" (id 1) (at 178.054 141.986 90))
+    (property "Value" "1k" (id 1) (at 178.054 141.986 90))
     (property "Footprint" "Capacitor_SMD:C_0603_1608Metric" (id 2) (at 178.054 147.574 90)
       (effects (font (size 1.27 1.27)) hide)
@@
       (effects (font (size 1.27 1.27)) (justify left))
     )
-    (property "Value" "C" (id 1) (at 186.436 150.8759 0)
+    (property "Value" "0.1uF" (id 1) (at 186.436 150.8759 0)
       (effects (font (size 1.27 1.27)) (justify left))
     )
@@
       (effects (font (size 1.27 1.27)) (justify left))
     )
-    (property "Value" "C" (id 1) (at 118.618 135.8899 0)
+    (property "Value" "0.1uF" (id 1) (at 118.618 135.8899 0)
       (effects (font (size 1.27 1.27)) (justify left))
     )
@@
     )
     (path "/18cf8238-146f-4d7e-a746-90549ffae207"
-      (reference "C9") (unit 1) (value "C") (footprint "Capacitor_SMD:C_0603_1608Metric")
+      (reference "C9") (unit 1) (value "0.1uF") (footprint "Capacitor_SMD:C_0603_1608Metric")
     )
     (path "/fd8de787-a23a-4e2e-aad7-1e5a28027dfa"
-      (reference "C10") (unit 1) (value "C") (footprint "Capacitor_SMD:C_0603_1608Metric")
+      (reference "C10") (unit 1) (value "0.1uF") (footprint "Capacitor_SMD:C_0603_1608Metric")
     )
     (path "/7c0895b6-15bb-4a54-9aa5-399b0ba067fe"
-      (reference "C11") (unit 1) (value "C") (footprint "Capacitor_SMD:C_0603_1608Metric")
+      (reference "C11") (unit 1) (value "0.1uF") (footprint "Capacitor_SMD:C_0603_1608Metric")
     )
     (path "/d7ac3cbc-803f-4363-a900-3cc2137bc2d8"
-      (reference "C12") (unit 1) (value "C") (footprint "Capacitor_SMD:C_0603_1608Metric")
+      (reference "C12") (unit 1) (value "0.1uF") (footprint "Capacitor_SMD:C_0603_1608Metric")
     )
     (path "/d67d0aec-122c-4a02-8c87-e3d73b1ddb3b"
@@
     )
     (path "/cfbd0ad0-03f8-4b91-aa03-6698bf547882"
-      (reference "R3") (unit 1) (value "R") (footprint "Capacitor_SMD:C_0603_1608Metric")
+      (reference "R3") (unit 1) (value "1k") (footprint "Capacitor_SMD:C_0603_1608Metric")
     )
     (path "/cbde98de-6ba1-421d-a2d1-83012244527c"
-      (reference "R4") (unit 1) (value "R") (footprint "Capacitor_SMD:C_0603_1608Metric")
+      (reference "R4") (unit 1) (value "1k") (footprint "Capacitor_SMD:C_0603_1608Metric")
     )
     (path "/9451f65d-5cb0-442a-87a1-191ad4ff98be"
-      (reference "R5") (unit 1) (value "R") (footprint "Capacitor_SMD:C_0603_1608Metric")
+      (reference "R5") (unit 1) (value "1k") (footprint "Capacitor_SMD:C_0603_1608Metric")
     )
     (path "/5d3bae2e-61ed-4d10-aa14-432570dd0c6d"
-      (reference "R6") (unit 1) (value "R") (footprint "Capacitor_SMD:C_0603_1608Metric")
+      (reference "R6") (unit 1) (value "1k") (footprint "Capacitor_SMD:C_0603_1608Metric")
     )
     (path "/43b59609-74fa-4505-9a82-8dfa3cda65ad"
